File: trinket.sch (KiCad schematic (older format))
At the start: 12 parts, among them SW1 POWER, U1 ATtiny414-SS, U2 MAN71A

Commit message: Revision 2 schematics
Connections:
- net at R1.2: now also U1.11 (PA1); no longer U1.10 (~RESET~/PA0)
- net at R2.2: now also U1.12 (PA2); no longer U1.11 (PA1)
- net at R3.2: now also U1.13 (PA3); no longer U1.12 (PA2)
- net at R4.2: now also U1.2 (PA4); no longer U1.13 (PA3)
- net at R5.2: now also U1.3 (PA5); no longer U1.2 (PA4)
- net at R6.2: now also U1.4 (PA6); no longer U1.3 (PA5)
- net at R7.2: now also U1.5 (PA7); no longer U1.4 (PA6)
- net RX: now reaches U1.6 (PB3)
- net TX: now reaches U1.7 (PB2)
- net PGM: now reaches U1.8 (PB1)
- net A: now reaches U2.1 (A)
- net A: now also R3.1; no longer R1.1
- net C: now reaches U2.10 (C)
- net C: now also R5.1; no longer R3.1
- net E: now reaches R7.1
- net E: now also U2.7 (E); no longer U2.11 (G)
- net B: now reaches U2.13 (B)
- net B: now also R4.1; no longer R2.1
- net D: now reaches R6.1
- net D: now also U2.8 (D); no longer U2.2 (F)
- new net F: R2.1, U2.2 (F)
- new net G: R1.1, U2.11 (G)
- new net UPDI: U1.10 (~RESET~/PA0)
- no-connect marks 0 -> 4
Other:
- moved on the sheet: C1, U2
